File: PCB/CapyController/CapyController/CapyController.kicad_sch (KiCad schematic)
At the start: 48 parts, among them J1 Conn_01x02, J10 Conn_01x04, J11 Conn_01x04, J12 Conn_01x04, J13 Conn_01x04, J14 Conn_01x02, J15 Conn_01x02, J16 Conn_01x04, J17 Conn_01x02, J18 Conn_01x04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

Commit message: Updated Both PCBs
Parts:
- J10, J11, J12, J13, J6, J7, J8, J9: footprint Connector_JST:JST_GH_BM04B-GHS-TBT_1x04-1MP_P1.25mm_Vertical -> Connector_JST:JST_PH_B4B-PH-K_1x04_P2.00mm_Vertical
- J2, J3: footprint Connector_JST:JST_GH_BM08B-GHS-TBT_1x08-1MP_P1.25mm_Vertical -> Connector_JST:JST_PH_B8B-PH-K_1x08_P2.00mm_Vertical
- J4, J5: footprint Connector_JST:JST_GH_BM04B-GHS-TBT_1x04-1MP_P1.25mm_Vertical -> Connector_JST:JST_PH_B5B-PH-K_1x05_P2.00mm_Vertical; symbol Connector_Generic:Conn_01x04 -> Connector_Generic:Conn_01x05
Connections:
- net GND: now also J4.5 (Pin_5), J5.5 (Pin_5)
Changed lines of the file:
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@@
 	)
 	(label "STPR_EN1"
-		(at 196.85 62.23 0)
+		(at 196.85 64.77 0)
 		(effects
 			(font
@@
 	)
 	(label "STPR_DIR1"
-		(at 196.85 59.69 0)
+		(at 196.85 62.23 0)
 		(effects
 			(font
@@
 	)
 	(label "STPR_EN2"
-		(at 219.71 62.23 0)
+		(at 219.71 64.77 0)
 		(effects
 			(font
@@
 	)
 	(label "STPR_DIR2"
-		(at 219.71 59.69 0)
+		(at 219.71 62.23 0)
 		(effects
 			(font
@@
 	)
 	(label "STPR_PUL1"
-		(at 196.85 57.15 0)
+		(at 196.85 59.69 0)
 		(effects
 			(font
@@
 	)
 	(label "STPR_PUL2"
-		(at 219.71 57.15 0)
+		(at 219.71 59.69 0)
 		(effects
 			(font
@@
 	)
 	(symbol
-		(lib_id "Connector_Generic:Conn_01x04")
+		(lib_id "Connector_Generic:Conn_01x05")
 		(at 191.77 62.23 180)
 		(unit 1)
@@
 			)
 		)
-		(property "Footprint" "Connector_JST:JST_GH_BM04B-GHS-TBT_1x04-1MP_P1.25mm_Vertical"
+		(property "Footprint" "Connector_JST:JST_PH_B5B-PH-K_1x05_P2.00mm_Vertical"
 			(at 191.77 62.23 0)
 			(effects
@@
 			)
 		)
-		(property "Description" "Generic connector, single row, 01x04, script generated (kicad-library-utils/schlib/autogen/connector/)"
+		(property "Description" "Generic connector, single row, 01x05, script generated (kicad-library-utils/schlib/autogen/connector/)"
 			(at 191.77 62.23 0)
 			(effects
@@
 		(pin "4"
 		)
+		(pin "5"
+		)
 		(instances
 			(project ""
@@
 			)
 		)
-		(property "Footprint" "Connector_JST:JST_GH_BM08B-GHS-TBT_1x08-1MP_P1.25mm_Vertical"
+		(property "Footprint" "Connector_JST:JST_PH_B8B-PH-K_1x08_P2.00mm_Vertical"
 			(at 220.98 36.83 0)
 			(effects
@@
 			)
 		)
-		(property "Footprint" "Connector_JST:JST_GH_BM04B-GHS-TBT_1x04-1MP_P1.25mm_Vertical"
+		(property "Footprint" "Connector_JST:JST_PH_B4B-PH-K_1x04_P2.00mm_Vertical"
 			(at 146.05 140.97 0)
 			(effects
@@
 			)
 		)
-		(property "Footprint" "Connector_JST:JST_GH_BM04B-GHS-TBT_1x04-1MP_P1.25mm_Vertical"
+		(property "Footprint" "Connector_JST:JST_PH_B4B-PH-K_1x04_P2.00mm_Vertical"
 			(at 72.39 140.97 0)
 			(effects
@@
 			)
 		)
-		(property "Footprint" "Connector_JST:JST_GH_BM08B-GHS-TBT_1x08-1MP_P1.25mm_Vertical"
+		(property "Footprint" "Connector_JST:JST_PH_B8B-PH-K_1x08_P2.00mm_Vertical"
 			(at 191.77 36.83 0)
 			(effects
@@
 	)
 	(symbol
-		(lib_id "Connector_Generic:Conn_01x04")
+		(lib_id "Connector_Generic:Conn_01x05")
 		(at 214.63 62.23 180)
 		(unit 1)
@@
 			)
 		)
-		(property "Footprint" "Connector_JST:JST_GH_BM04B-GHS-TBT_1x04-1MP_P1.25mm_Vertical"
+		(property "Footprint" "Connector_JST:JST_PH_B5B-PH-K_1x05_P2.00mm_Vertical"
 			(at 214.63 62.23 0)
 			(effects
@@
 			)
 		)
-		(property "Description" "Generic connector, single row, 01x04, script generated (kicad-library-utils/schlib/autogen/connector/)"
+		(property "Description" "Generic connector, single row, 01x05, script generated (kicad-library-utils/schlib/autogen/connector/)"
 			(at 214.63 62.23 0)
 			(effects
@@
 		(pin "4"
 		)
+		(pin "5"
+		)
 		(instances
 			(project "CapyController"
@@
 			)
 		)
-		(property "Footprint" "Connector_JST:JST_GH_BM04B-GHS-TBT_1x04-1MP_P1.25mm_Vertical"
+		(property "Footprint" "Connector_JST:JST_PH_B4B-PH-K_1x04_P2.00mm_Vertical"
 			(at 121.92 140.97 0)
 			(effects
@@
 			)
 		)
-		(property "Footprint" "Connector_JST:JST_GH_BM04B-GHS-TBT_1x04-1MP_P1.25mm_Vertical"
+		(property "Footprint" "Connector_JST:JST_PH_B4B-PH-K_1x04_P2.00mm_Vertical"
 			(at 96.52 172.72 0)
 			(effects
@@
 	(symbol
 		(lib_id "power:+5V")
-		(at 196.85 64.77 270)
+		(at 196.85 67.31 270)
 		(unit 1)
 		(exclude_from_sim no)
@@
 		(fields_autoplaced yes)
 		(property "Reference" "#PWR021"
-			(at 193.04 64.77 0)
+			(at 193.04 67.31 0)
 			(effects
 				(font
@@
 		)
 		(property "Value" "+3.3V"
-			(at 200.66 64.7699 90)
+			(at 200.66 67.3099 90)
 			(effects
 				(font
@@
 		)
 		(property "Footprint" ""
-			(at 196.85 64.77 0)
+			(at 196.85 67.31 0)
 			(effects
 				(font
@@
 		)
 		(property "Datasheet" ""
-			(at 196.85 64.77 0)
+			(at 196.85 67.31 0)
 			(effects
 				(font
@@
 		)
 		(property "Description" "Power symbol creates a global label with name \"+5V\""
-			(at 196.85 64.77 0)
+			(at 196.85 67.31 0)
 			(effects
 				(font
@@
 	(symbol
 		(lib_id "power:GND")
+		(at 219.71 57.15 90)
+		(unit 1)
+		(exclude_from_sim no)
+		(in_bom yes)
+		(on_board yes)
+		(dnp no)
+		(fields_autoplaced yes)
+		(property "Reference" "#PWR063"
+			(at 226.06 57.15 0)
+			(effects
+				(font
+					(size 1.27 1.27)
+				)
+				(hide yes)
+			)
+		)
+		(property "Value" "GND"
+			(at 223.52 57.1499 90)
+			(effects
+				(font
+					(size 1.27 1.27)
+				)
+				(justify right)
+			)
+		)
+		(property "Footprint" ""
+			(at 219.71 57.15 0)
+			(effects
+				(font
+					(size 1.27 1.27)
+				)
+				(hide yes)
+			)
+		)
+		(property "Datasheet" ""
+			(at 219.71 57.15 0)
+			(effects
+				(font
+					(size 1.27 1.27)
+				)
+				(hide yes)
+			)
+		)
+		(property "Description" "Power symbol creates a global label with name \"GND\" , ground"
+			(at 219.71 57.15 0)
+			(effects
+				(font
+					(size 1.27 1.27)
+				)
+				(hide yes)
+			)
+		)
+		(pin "1"
+		)
+		(instances
+			(project "CapyController"
+				(path "/9356d540-b2ec-4e7a-a3e1-4671cf217e36"
+					(reference "#PWR063")
+					(unit 1)
+				)
+			)
+		)
+	)
+	(symbol
+		(lib_id "power:GND")
 		(at 171.45 41.91 90)
 		(unit 1)
@@
 	(symbol
 		(lib_id "power:+5V")
-		(at 219.71 64.77 270)
+		(at 219.71 67.31 270)
 		(unit 1)
 		(exclude_from_sim no)
@@
 		(fields_autoplaced yes)
 		(property "Reference" "#PWR022"
-			(at 215.9 64.77 0)
+			(at 215.9 67.31 0)
 			(effects
 				(font
@@
 		)
 		(property "Value" "+3.3V"
-			(at 223.52 64.7699 90)
+			(at 223.52 67.3099 90)
 			(effects
 				(font
@@
 		)
 		(property "Footprint" ""
-			(at 219.71 64.77 0)
+			(at 219.71 67.31 0)
 			(effects
 				(font
@@
 		)
 		(property "Datasheet" ""
-			(at 219.71 64.77 0)
+			(at 219.71 67.31 0)
 			(effects
 				(font
@@
 		)
 		(property "Description" "Power symbol creates a global label with name \"+5V\""
-			(at 219.71 64.77 0)
+			(at 219.71 67.31 0)
 			(effects
 				(font
@@
 			)
 		)
-		(property "Footprint" "Connector_JST:JST_GH_BM04B-GHS-TBT_1x04-1MP_P1.25mm_Vertical"
+		(property "Footprint" "Connector_JST:JST_PH_B4B-PH-K_1x04_P2.00mm_Vertical"
 			(at 146.05 173.99 0)
 			(effects
@@
 	)
 	(symbol
+		(lib_id "power:GND")
+		(at 196.85 57.15 90)
+		(unit 1)
+		(exclude_from_sim no)
+		(in_bom yes)
+		(on_board yes)
+		(dnp no)
+		(fields_autoplaced yes)
+		(property "Reference" "#PWR062"
+			(at 203.2 57.15 0)
+			(effects
+				(font
+					(size 1.27 1.27)
+				)
+				(hide yes)
+			)
+		)
+		(property "Value" "GND"
+			(at 200.66 57.1499 90)
+			(effects
+				(font
+					(size 1.27 1.27)
+				)
+				(justify right)
+			)
+		)
+		(property "Footprint" ""
+			(at 196.85 57.15 0)
+			(effects
+				(font
+					(size 1.27 1.27)
+				)
+				(hide yes)
+			)
+		)
+		(property "Datasheet" ""
+			(at 196.85 57.15 0)
+			(effects
+				(font
+					(size 1.27 1.27)
+				)
+				(hide yes)
+			)
+		)
+		(property "Description" "Power symbol creates a global label with name \"GND\" , ground"
+			(at 196.85 57.15 0)
+			(effects
+				(font
+					(size 1.27 1.27)
+				)
+				(hide yes)
+			)
+		)
+		(pin "1"
+		)
+		(instances
+			(project "CapyController"
+				(path "/9356d540-b2ec-4e7a-a3e1-4671cf217e36"
+					(reference "#PWR062")
+					(unit 1)
+				)
+			)
+		)
+	)
+	(symbol
 		(lib_id "power:+5V")
 		(at 110.49 162.56 0)
@@
 			)
 		)
-		(property "Footprint" "Connector_JST:JST_GH_BM04B-GHS-TBT_1x04-1MP_P1.25mm_Vertical"
+		(property "Footprint" "Connector_JST:JST_PH_B4B-PH-K_1x04_P2.00mm_Vertical"
 			(at 120.65 172.72 0)
 			(effects
@@
 			)
 		)
-		(property "Footprint" "Connector_JST:JST_GH_BM04B-GHS-TBT_1x04-1MP_P1.25mm_Vertical"
+		(property "Footprint" "Connector_JST:JST_PH_B4B-PH-K_1x04_P2.00mm_Vertical"
 			(at 72.39 172.72 0)
 			(effects
@@
 			)
 		)
-		(property "Footprint" "Connector_JST:JST_GH_BM04B-GHS-TBT_1x04-1MP_P1.25mm_Vertical"
+		(property "Footprint" "Connector_JST:JST_PH_B4B-PH-K_1x04_P2.00mm_Vertical"
 			(at 96.52 140.97 0)
 			(effects

Commit message: Updated CapyPower
Parts:
- added C4: 47uF, Capacitor_SMD:C_1206_3216Metric, symbol Device:C
- added C5: 100nF, Capacitor_SMD:C_1206_3216Metric, symbol Device:C
- C1, C2, C3: footprint Capacitor_SMD:C_0402_1005Metric -> Capacitor_SMD:C_1206_3216Metric
Connections:
- net +3.3V: now also C4.2, C5.2
- net GND: now also C4.1, C5.1

Commit message: Updated CapyController
Other:
- company: (none) -> Imperial Planetary Roboics Lab
- title: (none) -> Capybara Rover Controller
Changed lines of the file:
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@@
 	(generator_version "9.0")
 	(paper "A4")
+	(title_block
+		(title "Capybara Rover Controller")
+		(date "2025-04-21")
+		(rev "2")
+		(company "Imperial Planetary Roboics Lab")
+	)
 	(text "I2C Multiplexer\n"
 		(exclude_from_sim no)
